Commit message: Updating simulation dialtone

File: oro_barrett_sim/test/idle.xacro (robot description, xacro)
@@ -1,4 +1,4 @@
 <?xml version="1.0"?>
-<robot xmlns:xacro="http://www.ros.org/wiki/xacro" name="sevenbot">
+<robot xmlns:xacro="http://www.ros.org/wiki/xacro" name="wam">
   <!-- Gazebo Plugin -->
   <gazebo>
@@ -15,5 +15,5 @@
   <include filename="$(find barrett_model)/models/wam_top.urdf.xacro"/>
   <!-- Root link is in the world frame-->
-  <link name = "world"/>
+  <link name="world"/>
   <xacro:wam_7dof prefix="wam" parent_link="world" xyz="0.02 0.46 1" rpy="0 0 0" />
 </robot>
